Commit message: added contact link and updated inertias

File: softleg_description/model/softleg_cart.urdf.xacro (robot description, xacro)
@@ -3,8 +3,7 @@
     <!-- Properties -->
     <xacro:property name="const_pi" value="3.1415926535897931"/>
-    <xacro:property name="cart_mass" value="0.0181"/>
-    <xacro:property name="base_mass" value="0.0256"/>
-    <xacro:property name="thigh_mass" value="0.0177"/>
-    <xacro:property name="calf_mass" value="0.0177"/>
+    <xacro:property name="base_mass" value="0.97245523"/>
+    <xacro:property name="thigh_mass" value="0.43578906"/>
+    <xacro:property name="calf_mass" value="0.076217499"/>
     <xacro:property name="velocity" value="100" />
     <xacro:property name="effort" value="100" />
@@ -93,5 +92,5 @@
             </collision>
         </link>
-        <!-- 1) Thigh link - rotates w.r.t base -->
+        <!-- 2) Thigh link - rotates w.r.t base -->
         <joint name="${name}_hip_joint" type="revolute">
             <origin xyz="0.255 0 0.07" rpy="${90 * const_pi / 180} 0 0"/>
@@ -141,5 +140,5 @@
             </collision>
         </link>
-        <!-- 1) Calf link - rotates w.r.t thigh -->
+        <!-- 3) Calf link - rotates w.r.t thigh -->
         <joint name="${name}_knee_joint" type="revolute">
             <origin xyz="0.175 0.0275 0" rpy="${90 * const_pi / 180} 0 0"/>
@@ -189,4 +188,15 @@
             </collision>
         </link>
+        <!-- 4) Contact link - Fixed -->
+        <joint name="${name}_contact_joint" type="fixed">
+            <origin xyz="0.185 0 -0.02" rpy="${90 * const_pi / 180} 0 0"/>
+            <parent link="${name}_calf_link"/>
+            <child link="${name}_contact_link"/>
+        </joint>
+        <link name="${name}_contact_link">
+            <inertial>
+                <xacro:insert_block name="really_negligible_inertia"/>
+            </inertial>
+        </link>
         <!-- Gazebo elements -->
         <xacro:softleg_gazebo name="${name}"/>

File: softleg_description/model/softleg_inertia.xacro (robot description, xacro)
@@ -5,23 +5,18 @@
     <xacro:property name="mm2tom2" value="0.000001"/>
     <!-- INERTIA MATRICES FOR LINKS (wrt frames in urdf inertial) -->
-    <!-- Cart -->
-    <xacro:macro name="cart_inertia">
-        <inertia ixx="${mm2tom2 * 4.4972}" iyy="${mm2tom2 * 1.8785}" izz="${mm2tom2 * 1.0468}"
-                 ixy="${mm2tom2 * -0.0012}" ixz="${mm2tom2 * -0.0027}" iyz="${mm2tom2 * 0.0005}"/>
-    </xacro:macro>
     <!-- Base -->
     <xacro:macro name="base_inertia">
-        <inertia ixx="${mm2tom2 * 3.1301}" iyy="${mm2tom2 * 12.3897}" izz="${mm2tom2 * 11.8654}"
-                 ixy="${mm2tom2 * -0.3627}" ixz="${mm2tom2 * 3.6816}" iyz="${mm2tom2 * 0.1283}"/>
+        <inertia ixx="${mm2tom2 * 1698.4399}" iyy="${mm2tom2 * 20148.638}" izz="${mm2tom2 * 19764.513}"
+                 ixy="${mm2tom2 * -983.90475}" ixz="${mm2tom2 * -1305.3791}" iyz="${mm2tom2 * 153.83174}"/>
     </xacro:macro>
     <!-- Thigh -->
     <xacro:macro name="thigh_inertia">
-        <inertia ixx="${mm2tom2 * 3.1301}" iyy="${mm2tom2 * 12.3897}" izz="${mm2tom2 * 11.8654}"
-                 ixy="${mm2tom2 * -0.3627}" ixz="${mm2tom2 * -3.6816}" iyz="${mm2tom2 * -0.1283}"/>
+        <inertia ixx="${mm2tom2 * 750.26891}" iyy="${mm2tom2 * 4575.9812}" izz="${mm2tom2 * 5105.9889}"
+                 ixy="${mm2tom2 * -1057.6540}" ixz="${mm2tom2 * 0.071507533}" iyz="${mm2tom2 * 0.32201257}"/>
     </xacro:macro>
     <!-- Calf -->
     <xacro:macro name="calf_inertia">
-        <inertia ixx="${mm2tom2 * 3.1301}" iyy="${mm2tom2 * 12.3897}" izz="${mm2tom2 * 11.8654}"
-                 ixy="${mm2tom2 * -0.3627}" ixz="${mm2tom2 * -3.6816}" iyz="${mm2tom2 * -0.1283}"/>
+        <inertia ixx="${mm2tom2 * 60.006429}" iyy="${mm2tom2 * 472.43319}" izz="${mm2tom2 * 520.49867}"
+                 ixy="${mm2tom2 * -119.84835e+02}" ixz="${mm2tom2 * 0.00036890095}" iyz="${mm2tom2 * 0.00012686113}"/>
     </xacro:macro>
     <!-- Simple cuboid -->
